Commit message: Rewrite LED hardware interface from GPIO to CAN
Replace GPIO sysfs-based LED control with CAN bus communication to match
the electrical team's actual hardware (CAN ID 0x170). Supports on/off,
red, and green commands via single-byte CAN frames.

Command interface encoding: 0.0=OFF, 1.0=ON, 2.0=RED, 3.0=GREEN.

File: src/description/ros2_control/drive/drive.led.ros2_control.xacro (robot description, xacro)
@@ -1,9 +1,10 @@
 <?xml version="1.0"?>
 <robot xmlns:xacro="http://www.ros.org/wiki/xacro">
-  <xacro:macro name="led_ros2_control" params="name gpio_pin default_state:=off">
+  <xacro:macro name="led_ros2_control" params="name can_interface:=can0 default_state:=off">
     <ros2_control name="${name}" type="system">
       <hardware>
         <plugin>led_ros2_control/LEDHardwareInterface</plugin>
-        <param name="gpio_pin">${gpio_pin}</param>
+        <param name="can_interface">${can_interface}</param>
+        <param name="can_id">0x170</param>
         <param name="default_state">${default_state}</param>
       </hardware>

File: src/description/urdf/athena_drive.urdf.xacro (robot description, xacro)
@@ -54,6 +54,6 @@
     <xacro:odrive_ros2_control name="odrive"/>
     <xacro:rmd_ros2_control name="rmd"/>
-    <!-- LED status indicator (GPIO-based) -->
-    <xacro:led_ros2_control name="status_led" gpio_pin="25"/>
+    <!-- LED status indicator (CAN-based) -->
+    <xacro:led_ros2_control name="status_led"/>
     <!-- Killswitch (CAN-based) -->
     <xacro:killswitch_ros2_control name="drive_killswitch"/>
