Commit message: feat(arm): belt coupling compensation for shoulder/elbow in RMD HWI
Shoulder and elbow share a belt; decouple joint state in read() and recouple commands in write() so all controllers see independent joints.

- Add coupled_mode, coupling_factor, driving_joint, coupled_joint in arm.rmd.ros2_control.xacro (defaults: coupled on, factor 1.0)
- Toggle via coupled_mode=false in xacro for legacy uncoupled behavior

Physical tuning (sign/factor) still required on hardware.

File: src/description/ros2_control/arm/arm.rmd.ros2_control.xacro (robot description, xacro)
@@ -1,5 +1,5 @@
 <?xml version="1.0"?>
 <robot xmlns:xacro="http://www.ros.org/wiki/xacro">
-  <xacro:macro name="rmd_ros2_control" params="name">
+  <xacro:macro name="rmd_ros2_control" params="name can_interface:=can0 coupled_mode:=true coupling_factor:=1.0">
     <ros2_control name="${name}" type="system">
       <hardware>
@@ -8,5 +8,9 @@
         <param name="logger_rate">5</param> <!-- Hz -->
         <param name="logger_state">0</param> <!-- 0 for off, 1 for on -->
-        <param name="can_interface">can0</param>
+        <param name="can_interface">${can_interface}</param>
+        <param name="coupled_mode">${coupled_mode}</param>
+        <param name="coupling_factor">${coupling_factor}</param>
+        <param name="driving_joint">shoulder_pitch</param>
+        <param name="coupled_joint">elbow_pitch</param>
       </hardware>
       <joint name="shoulder_pitch">
